File: pcb/FED3 v7.4/FED3.kicad_pcb (KiCad board)
At the start: 4 copper layers, 108 x 50 mm, 89 parts, among them IC1 MC74VHC1GT125, IC2 TB6612FNG, IC4 RTC PCF8523T, J1 Conn_02x03_Odd_Even, Q2 DMP2035U-7, SW1 Sw, SW2 SPST_TACT-KMR2, U1 ATSAMD21G18A, U2 MIC5504-3.3, U3 MCP73831T, X1 ClockXtal, X2 uXtal, X4 microsd, X5 JST-XH-02

Commit message: retomar sincronia PCB com main-branch @12Junho
Parts:
- AUX_I2C0: value TBD -> Qwiic
Other:
- board text added: ".2"
- board text removed: ".1"
Changed lines of the file:
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@@
 			(psa4output no)
 			(plot_black_and_white yes)
+			(plotinvisibletext no)
 			(sketchpadsonfab no)
 			(plotpadnumbers no)
@@
 		(sheetname "/controler stage/")
 		(sheetfile "controler stage.kicad_sch")
-		(attr exclude_from_pos_files)
 		(fp_line
 			(start -5.715 1.27)
@@
 		(sheetname "/controler stage/")
 		(sheetfile "controler stage.kicad_sch")
-		(attr through_hole exclude_from_pos_files)
+		(attr through_hole)
 		(fp_line
 			(start 3.92 -1.38)
@@
 			)
 		)
-		(property "Value" "TBD"
+		(property "Value" "Qwiic"
 			(at 0 3.3 180)
 			(unlocked yes)
@@
 			)
 		)
-		(property "OEPSPN" "TBD"
+		(property "OEPSPN" "OEPS070125"
 			(at 0 0 180)
 			(unlocked yes)
@@
 			)
 		)
-		(property "MPN" "n.a."
+		(property "MPN" "BM04B-SRSS-TB(LF)(SN)"
 			(at 0 0 180)
 			(unlocked yes)
@@
 		(sheetname "/")
 		(sheetfile "FED3.kicad_sch")
-		(attr exclude_from_pos_files)
 		(fp_line
 			(start 3.7 2.3575)
@@
 		(sheetname "/IOs Interface/")
 		(sheetfile "IOs Interface.kicad_sch")
-		(attr through_hole exclude_from_pos_files)
+		(attr through_hole)
 		(fp_line
 			(start -3.998 -0.004)
@@
 		(sheetname "/")
 		(sheetfile "FED3.kicad_sch")
-		(attr exclude_from_pos_files exclude_from_bom)
+		(attr exclude_from_bom)
 		(fp_line
 			(start -6.35 -0.635)
@@
 	)
 	(gr_text "Qwiic"
-		(at 127.92 118.82 0)
+		(at 128.08 119.06 0)
 		(layer "F.SilkS")
 		(effects
@@
 	)
 	(gr_text "STEMMA QT"
-		(at 127.92 117.29 0)
+		(at 128.08 117.53 0)
 		(layer "F.SilkS")
 		(effects
@@
 	)
 	(gr_text "CHARGING"
-		(at 199.704163 105.423767 90)
+		(at 199.95 105.41 90)
 		(layer "F.SilkS")
 		(effects
@@
 		)
 	)
-	(gr_text ".1"
+	(gr_text ".2"
 		(at 110.7 96.628 0)
 		(layer "F.SilkS")
@@
 			(font
 				(size 1.64084 1.64084)
-				(thickness 0.28956)
+				(thickness 0.328168)
+				(bold yes)
 			)
 			(justify left bottom)
@@
 		(effects
 			(font
-				(size 1 1)
+				(size 0.8 1)
 				(thickness 0.2)
 			)
