File: pcb/FED3 v7.4/FED3.kicad_sch (KiCad schematic)
At the start: 27 parts, among them IC2 TB6612FNG, SW1 Sw, U2 MIC5504-3.3, U3 MCP73831T, X5 JST-XH-02

Commit message: last tunnings
- Top & Bottom Fabrication Layers tuned
- generated Gerbers&Drills files
- generated P&P & BOM files
Parts:
- L2, R19, R7: now in the parts list
Changed lines of the file:
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@@
 		(unit 1)
 		(exclude_from_sim no)
-		(in_bom no)
+		(in_bom yes)
 		(on_board yes)
 		(dnp yes)
@@
 		(unit 1)
 		(exclude_from_sim no)
-		(in_bom no)
+		(in_bom yes)
 		(on_board yes)
 		(dnp yes)
@@
 		(unit 1)
 		(exclude_from_sim no)
-		(in_bom no)
+		(in_bom yes)
 		(on_board yes)
 		(dnp yes)

Commit message: 'ultima versão revista; não em tunning com a versão oficial /Kravitz/FED3
Parts:
- IC2: MPN TB6612FNG,C,8,EL -> TB6612FNG,C,8,EL
- MOTOR0: now in the parts list
- SW1: MPN SSSS811101 -> SSSS811101
Changed lines of the file:
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@@
 			)
 		)
-		(property "MPN" "SSSS811101 "
+		(property "MPN" "SSSS811101"
 			(at 102.87 40.64 0)
 			(effects
@@
 			)
 		)
-		(property "MPN" "TB6612FNG,C,8,EL "
+		(property "MPN" "TB6612FNG,C,8,EL"
 			(at 204.47 124.46 0)
 			(effects
@@
 		(unit 1)
 		(exclude_from_sim no)
-		(in_bom no)
-		(on_board yes)
-		(dnp no)
+		(in_bom yes)
+		(on_board yes)
+		(dnp no)
