File: pcb/FED3 tester projects/FED3 tester/FED3 tester-backups/DUT.kicad_sch (KiCad schematic)
At the start: 68 parts, among them J3 6pin_hd, J4 Conn_02x03_Odd_Even, J5 MotorCkeck1, J6 MotorCkeck2, J7 Conn_01x02_Socket, K1 Relay SPDT, K2 Relay SPDT, K3 Relay SPDT, Q2 ???????, Q3 DMN63D8L-7, Q4 DMN63D8L-7, Q5 DMN63D8L-7, Q6 DMN63D8L-7, U6 THS4281, U7 THS4281, U8 THS4281, U9 ZXCT1082

Commit message: FED3 tester project
.commit para sincronia
.ainda longe do final
Parts:
- removed Q2: ???????, Package_TO_SOT_SMD:SOT-23, symbol Transistor_FET:BSS84
- removed Q3: DMN63D8L-7, Package_TO_SOT_SMD:SOT-23, symbol Transistor_FET:IRLML2060
- removed R27, R29, R32: 1.2K, Resistor_SMD:R_0402_1005Metric, symbol Device:R_US
- added C20: 100nF, Capacitor_SMD:C_0402_1005Metric, symbol Device:C_Small
- added C22, C23: 15nF, Capacitor_SMD:C_0402_1005Metric, symbol Device:C_Small
- added R17, R19, R20: 10k, Resistor_SMD:R_0402_1005Metric, symbol Device:R_US
- added R23: 5.1k, Resistor_SMD:R_0402_1005Metric, symbol Device:R_US
- added R49: 1k, Resistor_SMD:R_0402_1005Metric, symbol Device:R_US
- added TP11: GND, FED3_PCBLib:Pin_D1.75mm, symbol Connector:TestPoint
- added U6: THS4281, Package_TO_SOT_SMD:SOT-23-5, symbol FED3 SymbLib:THS4281DBVT
- renumbered C31 to C14, C32 to C15, C33 to C16, C34 to C17, C35 to C18, C36 to C19, C37 to C21, C38 to C24, C39 to C25, D10 to D1, D12 to D10, D11 to D8, J3 to J2, J4 to J3, J5 to J4, J6 to J5, Q4 to Q1, Q5 to Q3, Q6 to Q4, R20 to R10, R21 to R11, R22 to R12, R23 to R13, R24 to R14, R25 to R15, R26 to R16, R28 to R18, R30 to R21, R31 to R22, R33 to R24, R34 to R25, R37 to R26, R38 to R27, R39 to R28, R41 to R29, R44 to R30, R40 to R43, R42 to R44, R36 to R45, R43 to R46, R45 to R47, R46 to R48, R35 to R50, R19 to R9, TP11 to TP12, TP12 to TP13, TP8 to TP4, TP6 to TP5, TP7 to TP6, TP4 to TP7, TP5 to TP8, U6 to U4, U7 to U5, U8 to U7, U9 to U8
Connections:
- net +3V3: now also C20.1, U6.5 (V+)
- net GND: now also C20.2, C22.2, C23.2, R23.1, U6.2 (V-)
- net DUT_SWCLK renamed SWCLK
- net DUT_SWDIO renamed SWDIO
- net DUT_~{RESET} renamed ~{RESET}
- net VUSB_out renamed VUSBtest
- net VUSBtest: now also R17.2
- new net: R17.1, R23.2, U6.3 (+)
- new net: R19.1, U6.1, U6.4 (-)
- new net: C22.1, R19.2, R20.1
- new net: R49.2, TP11.1
- new net VUSB_check: C23.1, R20.2
- new net ~{RESET}_Test: R49.1
Other:
- moved on the sheet: TP4
