File: pcb/FED3 tester projects/FED3 tester/FED3 tester-backups/FED3 tester.kicad_sch (KiCad schematic)
At the start: 33 parts, among them J1 USB4105-GF-A, U1 FT232RL, U2 LP5907MFX-3.3, U3 LP5907MFX-3.3, U4 TPS79301DBVRG4

Commit message: FED3 tester project
.commit para sincronia
.ainda longe do final
Parts:
- removed C10, C13: 100nF, Capacitor_SMD:C_0402_1005Metric, symbol Device:C_Small
- removed C11: 2.2uF, Capacitor_SMD:C_0603_1608Metric, symbol Device:C_Small
- removed C12: 4.7uF, Capacitor_SMD:C_0603_1608Metric, symbol Device:C_Small
- removed U3: LP5907MFX-3.3, Package_TO_SOT_SMD:SOT-23-5, symbol Regulator_Linear:LP5907MFX-3.3
- renumbered C14 to C10, C15 to C11, C16 to C12, C17 to C13, U4 to U3
