File: pcb/FED3 tester projects/FED3 tester/FED3 tester-backups/main core.kicad_sch (KiCad schematic)
At the start: 33 parts, among them J1 USB4105-GF-A, U1 FT232RL, U2 LP5907MFX-3.3, U3 LP5907MFX-3.3, U4 TPS79301DBVRG4

Commit message: FED3 tester project
.commit para sincronia
.ainda longe do final
Parts:
- removed C1, C10, C13, C16, C2, C3, C5, C6, C9: 100nF, Capacitor_SMD:C_0402_1005Metric, symbol Device:C_Small
- removed C11, C7: 2.2uF, Capacitor_SMD:C_0603_1608Metric, symbol Device:C_Small
- removed C12, C15, C8: 4.7uF, Capacitor_SMD:C_0603_1608Metric, symbol Device:C_Small
- removed C14: 15pF, Capacitor_SMD:C_0603_1608Metric, symbol Device:C_Small
- removed C17: 10nF, Capacitor_SMD:C_0402_1005Metric, symbol Device:C_Small
- removed C4: 4.7nF, Capacitor_SMD:C_0402_1005Metric, symbol Device:C_Small
- removed J1: USB4105-GF-A, Connector_USB:USB_C_Receptacle_GCT_USB4105-xx-A_16P_TopMnt_Horizontal, symbol Connector:USB_C_Receptacle_USB2.0_16P
- removed L1, L2: 40R@100MHz, Resistor_SMD:R_0805_2012Metric, symbol Device:R
- removed R1, R3: 5.1k, Resistor_SMD:R_0402_1005Metric, symbol Device:R_US
- removed R2: 10k, Resistor_SMD:R_0402_1005Metric, symbol Device:R_US
- removed R4, R5: 27R, Resistor_SMD:R_0402_1005Metric, symbol Device:R_Small_US
- removed R6: 1M, Resistor_SMD:R_0402_1005Metric, symbol Device:R_US
- removed R7: 61.2k, Resistor_SMD:R_0402_1005Metric, symbol Device:R_US
- removed R8: 30.1k, Resistor_SMD:R_0603_1608Metric, symbol Device:R_US
- removed TP1: GND, Connector_PinHeader_2.54mm:PinHeader_1x01_P2.54mm_Vertical, symbol Connector:TestPoint
- removed U1: FT232RL, Package_SO:SSOP-28_5.3x10.2mm_P0.65mm, symbol Interface_USB:FT232RL
- removed U2, U3: LP5907MFX-3.3, Package_TO_SOT_SMD:SOT-23-5, symbol Regulator_Linear:LP5907MFX-3.3
- removed U4: TPS79301DBVRG4, Package_TO_SOT_SMD:SOT-23-6, symbol Regulator_Linear:TPS79301-EP
- added BZ1: Buzzer, FED3_PCBLib:SMT-0540-T-9-R Buzzer, symbol Device:Buzzer
- added C26, C27, C28, C29, C30, C31, C32, C33, C34, C35: 100nF, Capacitor_SMD:C_0402_1005Metric, symbol Device:C_Small
- added D2: 1N4148, Diode_SMD:D_SOD-123, symbol Diode:1N4148W
- added D3, D4, D5, D6, D7: Green LED, LED_SMD:LED_0603_1608Metric, symbol Device:LED
- added J6: Conn_02x03_Odd_Even, Connector_PinHeader_2.54mm:PinHeader_2x03_P2.54mm_Vertical, symbol Connector_Generic:Conn_02x03_Odd_Even
- added OSC1: 32MHz, FED3_PCBLib:OSC, symbol FED3 SymbLib:OSC_1
- added Q2: DMN63D8L-7, Package_TO_SOT_SMD:SOT-23, symbol Transistor_FET:IRLML2060
- added R36: 100R, Resistor_SMD:R_0402_1005Metric, symbol Device:R_Small_US
- added R37: 10k, Resistor_SMD:R_0402_1005Metric, symbol Device:R_US
- added R38, R39, R40, R41: 330R, Resistor_SMD:R_0402_1005Metric, symbol Device:R_US
- added R42: 560R, Resistor_SMD:R_0402_1005Metric, symbol Device:R_US
- added SW1, SW2, SW3, SW4, SW5: SW_SPST, Button_Switch_SMD:SW_SPST_TL3305B, symbol Switch:SW_Push
- added U9: ATXMEGA32A4U-MH, Package_DFN_QFN:QFN-44-1EP_7x7mm_P0.5mm_EP5.2x5.2mm, symbol FED3 SymbLib:ATXMEGA32A4U
Connections:
- net +3V3: now also C27.1, C28.1, C29.1, C30.1, C35.1, J6.2 (Pin_2), OSC1.4 (VDD), R36.1, U9.19 (VCC), U9.31 (VCC), U9.39 (AVCC), U9.9 (VCC)
- net GND: now also C26.2, C27.2, C28.2, C29.2, C30.2, C31.2, C32.2, C33.2, C34.2, C35.2, D3.1 (K), D4.1 (K), D5.1 (K), D6.1 (K), D7.1 (K), J6.6 (Pin_6), OSC1.2 (GND), Q2.2 (S), R37.1, SW1.1, SW2.1, SW3.1, SW4.1, SW5.1, U9.18 (GND), U9.30 (GND), U9.38 (GND), U9.45 (GND), U9.8 (GND)
- new net: D3.2 (A), R38.1
- new net: D4.2 (A), R39.1
- new net: D5.2 (A), R40.1
- new net: D7.2 (A), R42.1
- new net: BZ1.1 (+), D2.1 (K), R36.2
- new net: BZ1.2 (-), D2.2 (A), Q2.3 (D)
- new net: D6.2 (A), R41.1
- new net +3V3test_check: U9.43 (PA3/ADC3)
- new net ADC Bat_I: U9.3 (PA7/ADC7/AC0-OUT)
- new net Buzzer: Q2.1 (G), R37.2, U9.17 (PC7/SCK/TXD1/CLCKO/EVO)
- new net Buzzer_NOK: C32.1, SW3.2, U9.22 (PD2/OC0C/RXD0)
- new net Buzzer_OK: C31.1, SW2.2, U9.21 (PD1/OC0B/XCK0)
- new net FTDI_CTS: U9.29 (PE1/OC0B/XCK0/SCL)
- new net FTDI_RTS: U9.28 (PE0/OC0A/SDA)
- new net FTDI_RXD: U9.33 (PE3/OC0D/TXD0)
- new net FTDI_TXD: U9.32 (PE2/OC0C/RXD0)
- new net I ON/OFF Test: U9.7 (PB3/ADC11/DAC1)
- new net LED#1: R39.2, U9.10 (PC0/OC0A/SDA)
- new net LED#2: R40.2, U9.11 (PC1/OC0B/XCK0/SCL)
- new net LED#3: R41.2, U9.12 (PC2/OC0C/RXD0)
- new net LED#4: R42.2, U9.13 (PC3/OC0D/TXD0)
- new net LED_CHRG: U9.44 (PA4/ADC4)
- new net LED_GREEN: U9.2 (PA6/ADC6)
- new net Motor_NOK: C34.1, SW5.2, U9.24 (PD4/OC1A/~{SS})
- new net Motor_OK: C33.1, SW4.2, U9.23 (PD3/OC0D/TXD0)
- new net OSC: OSC1.3 (OUT), U9.37 (PR1/XTAL1)
- new net PDI_CLOCK: J6.5 (Pin_5), U9.35 (~{RESET}/PDI_CLOCK)
- new net PDI_DATA: J6.1 (Pin_1), U9.34 (PDI_DATA)
- new net POWER_EN: U9.27 (PD7/TXD1/SCK/CLCKO/D+)
- new net RED_LED: U9.1 (PA5/ADC5)
- new net Relay_ThermalPin: U9.5 (PB1/ADC9)
- new net Relay_VBattest: U9.4 (PB0/ADC8/AREF)
- new net START_SW: C26.1, SW1.2, U9.20 (PD0/OC0A)
- new net STATE_LED: R38.2, U9.36 (PR0/XTAL2)
- new net VBattest_check: U9.40 (PA0/ADC0/AREF)
- new net VUSB_check: U9.41 (PA1/ADC1)
- new net VccRGB_check: U9.42 (PA2/ADC2)
- new net ~{RESET}_Test: U9.26 (PD6/RXD1/MISO/D-)
- no-connect marks 13 -> 8
Other:
- removed sheet main core
- added sheet DUT stage (DUT.kicad_sch)
- title: FED3 Test Board -> (none)
