File: pcb/FED3 tester projects/FED3 tester/FED3 tester.kicad_pcb (KiCad board)
At the start: 4 copper layers, 108 x 134.4 mm, 164 parts, among them J1 USB4105-GF-A, J2 Conn_02x03_Odd_Even, J3 6pin_hd, J4 Conn_02x03_Odd_Even, J5 MotorCkeck1, J6 MotorCkeck2, J7 Conn_01x02_Socket, K1 Relay SPDT, K2 Relay SPDT, K3 Relay SPDT, Q1 DMN63D8L-7, Q2 ???????, Q3 DMN63D8L-7, Q4 DMN63D8L-7, Q5 DMN63D8L-7, Q6 DMN63D8L-7, SW1 SW_SPST, SW2 SW_SPST, SW3 SW_SPST, SW4 SW_SPST, SW5 SW_SPST, SW6 SW_SPST, SW7 SW_SPST, SW8 SW_SPST, SW9 SW_SPST, U1 FT232RL, U2 LP5907MFX-3.3, U3 LP5907MFX-3.3, U4 TPS73801DCQR, U5 ATXMEGA32A4U-MH, U6 THS4281, U7 THS4281, U8 THS4281, U9 ZXCT1082

Commit message: FED3 tester rev.B & FED3 tester support rev.B
-rev.B para 1ª revisão do Filipe
Parts:
- removed the ? at (111.1, 60.6)
- removed the ? at (67.2, 100.7)
- removed the ? at (63.5, 30.6)
- removed the ? at (66.7, 43.2)
- removed the ? at (112.8, 84.4)
- removed the ? at (65.4, 69.2)
- removed the ? at (154.2, 100.7)
- removed the ? at (154.4, 79.6)
- removed the ? at (154.2, 153.0)
- removed the ? at (158.0, 30.6)
- removed the ? at (67.2, 153.0)
- removed @HOLE0: , 
- removed the @HOLE6 at (140.7, 60.2)
- removed the D2 at (110.5, 103.1)
- removed the R10 at (106.3, 103.1)
- added ?: MechHole_7mm, FED3_PCBLib:MechHole_7mm, F.Cu at (111.1, 60.6)
- added ?: MechHole_7mm, FED3_PCBLib:MechHole_7mm, F.Cu at (154.2, 153.0)
- added ?: MechHole_7mm, FED3_PCBLib:MechHole_7mm, F.Cu at (67.2, 153.0)
- added ?: MechHole_7mm, FED3_PCBLib:MechHole_7mm, F.Cu at (67.2, 100.7)
- added ?: MechHole_7mm, FED3_PCBLib:MechHole_7mm, F.Cu at (158.0, 30.6)
- added ?: MechHole_7mm, FED3_PCBLib:MechHole_7mm, F.Cu at (63.5, 30.6)
- added ?: MechHole_7mm, FED3_PCBLib:MechHole_7mm, F.Cu at (154.2, 100.7)
- added @HOLE6: , FED3_PCBLib:MechHole_6.05mm, F.Cu at (144.2, 34.2)
- added @HOLE6: , FED3_PCBLib:MechHole_6.05mm, F.Cu at (140.7, 60.2)
- added @HOLE6: , FED3_PCBLib:MechHole_6.05mm, F.Cu at (66.7, 43.2)
- added Ref**: Val**, FED3_PCBLib:MechHole_2.95mm, F.Cu at (154.4, 79.6)
- added Ref**: Val**, FED3_PCBLib:MechHole_2.95mm, F.Cu at (112.8, 84.4)
- added Ref**: Val**, FED3_PCBLib:MechHole_2.95mm, F.Cu at (153.1, 142.8)
- added Ref**: Val**, FED3_PCBLib:MechHole_2.95mm, F.Cu at (65.4, 69.2)
- added Ref**: Val**, FED3_PCBLib:MechHole_2.95mm, F.Cu at (112.5, 142.8)
- Q2: value ??????? -> PMF170XP,115; footprint Package_TO_SOT_SMD:SOT-23 -> Package_TO_SOT_SMD:SOT-323_SC-70
- moved C10 75.1 mm to (109.3, 41.9), turned to 90 degrees
- moved C11 69.7 mm to (111.5, 41.6), turned to 90 degrees
- moved U3 67.9 mm to (115.4, 41.5)
- moved C13 63.2 mm to (121.0, 41.1), turned to -90 degrees
- moved C12 61.7 mm to (119.0, 41.4), turned to -90 degrees
- moved C16 38.4 mm to (114.0, 94.2)
- moved D6 18.5 mm to (71.0, 78.8), turned to 0 degrees
- moved R14 18.0 mm to (71.3, 76.3), turned to 180 degrees
- moved C15 16.8 mm to (76.4, 90.7), turned to 0 degrees
- moved R8 15.9 mm to (79.0, 84.1)
- moved C14 15.7 mm to (82.2, 85.9)
- moved R34 15.5 mm to (114.4, 50.1), turned to 180 degrees
- moved R7 15.4 mm to (79.0, 86.8)
- moved U4 15.4 mm to (73.3, 86.1)
- moved R38 10.9 mm to (67.5, 47.9), turned to 90 degrees
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- renumbered C15 to C14, C16 to C15, C17 to C16, C18 to C17, C19 to C18, C20 to C19, C21 to C20, C22 to C21, C23 to C22, C24 to C23, C25 to C24, C26 to C25, C27 to C26, C28 to C27, C29 to C28, C30 to C29, C31 to C30, C32 to C31, C33 to C32, C34 to C33, C35 to C34, C36 to C35, C37 to C36, C38 to C37, D11 to D10, D12 to D11, D3 to D2, D4 to D3, D5 to D4, D6 to D5, D7 to D6, D8 to D7, D9 to D8, D10 to D9, R11 to R10, R12 to R11, R13 to R12, R14 to R13, R15 to R14, R16 to R15, R17 to R16, R18 to R17, R19 to R18, R20 to R19, R21 to R20, R22 to R21, R23 to R22, R24 to R23, R25 to R24, R26 to R25, R27 to R26, R28 to R27, R29 to R28, R30 to R29, R31 to R30, R32 to R31, R33 to R32, R34 to R33, R35 to R34, R36 to R35, R37 to R36, R38 to R37, R39 to R38, R40 to R39, R41 to R40, R42 to R41, R43 to R42, R44 to R43, R45 to R44, R46 to R45, R47 to R46, R48 to R47
Connections:
- net /main core/DUT stage/+3V3test renamed /main core/DUT stage/+3V3_DUT
- net /main core/DUT stage/DUT_SWCLK renamed /main core/DUT stage/SWCLK_DUT
- net /main core/DUT stage/DUT_SWDIO renamed /main core/DUT stage/SWDIO_DUT
- net /main core/DUT stage/ExtVUSB renamed /main core/DUT stage/ExtVUSB_DUT
- net /main core/DUT stage/ThermalPin renamed /main core/DUT stage/ThermalPin_DUT
- net /main core/DUT stage/VBattest renamed /main core/DUT stage/VBatt_DUT
- net /main core/DUT stage/VUSB_out renamed /main core/DUT stage/VUSB_DUT
- net /main core/DUT stage/VccRGB renamed /main core/DUT stage/VccRGB_DUT
- net /main core/I ON/OFF Test renamed /main core/I_ON/OFF_Test
- R10 pad 2: /main core/LED#3 -> /main core/LED#2
- R11 pad 2: /main core/LED#4 -> /main core/LED#3
- R12 pad 2: /main core/LED#5 -> /main core/LED#4
- U5 pad 14: /main core/LED#5 -> /main core/VUSB_2DUT
- U5 pad 42: /main core/VUSB_2DUT -> /main core/VccRGB_check
Routing:
- net USB+5V: track 90.3 -> 264.5 mm, vias 3 -> 7
- net GND: track 63.5 -> 217.1 mm, vias 47 -> 82
- net /main core/Buzzer_NOK: track 0.00 -> 127.0 mm, vias 0 -> 3
- net +3V3: track 487.0 -> 595.8 mm, vias 25 -> 23
- net /main core/PASS: track 0.00 -> 103.6 mm, vias 0 -> 2
- net /main core/FAIL: track 0.00 -> 99.8 mm, vias 0 -> 2
- net /main core/Buzzer_OK: track 0.00 -> 94.4 mm, vias 0 -> 2
- net /main core/RGBW_NOK: track 19.8 -> 96.2 mm, vias 1 -> 2
- net /main core/Motor_NOK: track 4.18 -> 79.4 mm, vias 0 -> 3
- net /main core/Prog_OK: track 36.3 -> 99.1 mm
- net /main core/VBattest_check: track 93.7 -> 35.0 mm, vias 5 -> 3
- net RELAY+5V: track 84.3 -> 142.4 mm
- net /main core/RGBW_OK: track 16.1 -> 71.3 mm, vias 1 -> 2
- net /main core/VUSB_2DUT: track 0.00 -> 54.7 mm, vias 0 -> 2
- net /main core/Motor_OK: track 0.00 -> 54.7 mm, vias 0 -> 2
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- added copper zone on B.Cu, net GND
- added copper zone on In1.Cu, net GND
- added copper zone on In2.Cu, net GND
Other:
- board text removed: "READY 2PROGRAM"
- board text removed: "~{RESET}"
